File: pcb/cad/Fonte-de-corrente-SWLS_V0/Fonte-de-corrente-SWLS_V0.kicad_sch (KiCad schematic)
At the start: 32 parts, among them J2 LEMO FFA.0S, J3 LEMO FFA.0S, J4 Barrel_Jack_Switch, SW1 SW_DIP_x01, U1 LM78L05, U2 LT3080xST, U3 LT3092xST, U4 LT3092xST, U5 74AHC1G04, U6 TS5A21366, U7 TS5A21366, U8 TS5A21366, U9 TS5A21366

Commit message: Atualização do layout de PCB
Connections:
- net 1mADC_CH1: now also U7.2 (COM1), U8.6 (COM2); no longer U7.1 (NO1), U8.5 (NO2)
- net 1mADC_CH2: now also U6.2 (COM1), U9.6 (COM2); no longer U6.1 (NO1), U9.1 (NO1)
- net CH1+: now also U7.1 (NO1); no longer U7.2 (COM1)
- net CH1-: now also U8.5 (NO2); no longer U8.6 (COM2)
- net CH2+: now also U6.1 (NO1), U9.2 (COM1); no longer U6.2 (COM1), U6.6 (COM2)
- net CH2-: now also U6.6 (COM2), U9.5 (NO2); no longer U9.2 (COM1), U9.6 (COM2)
- net GND: now also U9.1 (NO1); no longer U9.5 (NO2)
- net IN: now also R3.2, SW1.2, U6.3 (IN2); no longer U9.3 (IN2)
- net ~{IN}: now also U9.3 (IN2); no longer U6.3 (IN2)
Changed lines of the file:
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@@
   (junction (at 54.61 41.91) (diameter 0) (color 0 0 0 0)
   )
+  (junction (at 134.62 154.94) (diameter 0) (color 0 0 0 0)
+  )
   (junction (at 39.37 95.25) (diameter 0) (color 0 0 0 0)
   )
@@
   (junction (at 50.8 49.53) (diameter 0) (color 0 0 0 0)
   )
-  (junction (at 134.62 156.21) (diameter 0) (color 0 0 0 0)
+  (junction (at 116.84 154.94) (diameter 0) (color 0 0 0 0)
   )
   (junction (at 151.13 46.99) (diameter 0) (color 0 0 0 0)
@@
     (stroke (width 0) (type default))
   )
-  (wire (pts (xy 116.84 156.21) (xy 134.62 156.21))
+  (wire (pts (xy 116.84 154.94) (xy 134.62 154.94))
     (stroke (width 0) (type default))
   )
@@
     (stroke (width 0) (type default))
   )
-  (wire (pts (xy 134.62 156.21) (xy 165.1 156.21))
+  (wire (pts (xy 134.62 154.94) (xy 165.1 154.94))
     (stroke (width 0) (type default))
   )
@@
     (stroke (width 0) (type default))
   )
-  (wire (pts (xy 134.62 156.21) (xy 134.62 180.34))
+  (wire (pts (xy 134.62 154.94) (xy 134.62 180.34))
     (stroke (width 0) (type default))
   )
@@
     (effects (font (size 2 2)) (justify left bottom))
   )
-  (label "CH1+" (at 224.79 39.37 0) (fields_autoplaced)
-    (effects (font (size 1.27 1.27)) (justify left bottom))
-  )
-  (label "1mADC_CH2" (at 196.85 86.36 180) (fields_autoplaced)
-    (effects (font (size 1.27 1.27)) (justify right bottom))
+  (label "CH1-" (at 224.79 52.07 0) (fields_autoplaced)
+    (effects (font (size 1.27 1.27)) (justify left bottom))
   )
   (label "5V_REG" (at 128.27 69.85 0) (fields_autoplaced)
     (effects (font (size 1.27 1.27)) (justify left bottom))
   )
+  (label "CH2-" (at 246.38 99.06 180) (fields_autoplaced)
+    (effects (font (size 1.27 1.27)) (justify right bottom))
+  )
+  (label "CH1-" (at 245.11 50.8 180) (fields_autoplaced)
+    (effects (font (size 1.27 1.27)) (justify right bottom))
+  )
   (label "VIN" (at 62.23 41.91 0) (fields_autoplaced)
     (effects (font (size 1.27 1.27)) (justify left bottom))
   )
-  (label "~{IN}" (at 196.85 104.14 180) (fields_autoplaced)
-    (effects (font (size 1.27 1.27)) (justify right bottom))
-  )
   (label "IN" (at 199.39 41.91 180) (fields_autoplaced)
     (effects (font (size 1.27 1.27)) (justify right bottom))
@@
     (effects (font (size 1.27 1.27)) (justify right bottom))
   )
+  (label "CH2+" (at 196.85 86.36 180) (fields_autoplaced)
+    (effects (font (size 1.27 1.27)) (justify right bottom))
+  )
+  (label "IN" (at 196.85 104.14 180) (fields_autoplaced)
+    (effects (font (size 1.27 1.27)) (justify right bottom))
+  )
   (label "~{IN}" (at 245.11 43.18 180) (fields_autoplaced)
     (effects (font (size 1.27 1.27)) (justify right bottom))
@@
     (effects (font (size 1.27 1.27)) (justify left bottom))
   )
-  (label "CH2-" (at 271.78 88.9 0) (fields_autoplaced)
-    (effects (font (size 1.27 1.27)) (justify left bottom))
-  )
-  (label "IN" (at 246.38 104.14 180) (fields_autoplaced)
-    (effects (font (size 1.27 1.27)) (justify right bottom))
-  )
   (label "~{IN}" (at 163.83 180.34 0) (fields_autoplaced)
     (effects (font (size 1.27 1.27)) (justify left bottom))
   )
+  (label "CH2-" (at 222.25 101.6 0) (fields_autoplaced)
+    (effects (font (size 1.27 1.27)) (justify left bottom))
+  )
+  (label "1mADC_CH1" (at 270.51 53.34 0) (fields_autoplaced)
+    (effects (font (size 1.27 1.27)) (justify left bottom))
+  )
   (label "CH1+" (at 222.25 142.24 0) (fields_autoplaced)
     (effects (font (size 1.27 1.27)) (justify left bottom))
   )
-  (label "1mADC_CH1" (at 245.11 50.8 180) (fields_autoplaced)
-    (effects (font (size 1.27 1.27)) (justify right bottom))
-  )
-  (label "1mADC_CH1" (at 199.39 36.83 180) (fields_autoplaced)
+  (label "1mADC_CH1" (at 224.79 39.37 0) (fields_autoplaced)
+    (effects (font (size 1.27 1.27)) (justify left bottom))
+  )
+  (label "CH1+" (at 199.39 36.83 180) (fields_autoplaced)
     (effects (font (size 1.27 1.27)) (justify right bottom))
   )
@@
     (effects (font (size 1.27 1.27)) (justify left bottom))
   )
-  (label "CH2-" (at 271.78 101.6 0) (fields_autoplaced)
+  (label "1mADC_CH2" (at 271.78 101.6 0) (fields_autoplaced)
     (effects (font (size 1.27 1.27)) (justify left bottom))
   )
@@
     (effects (font (size 1.27 1.27)) (justify right bottom))
   )
-  (label "1mADC_CH2" (at 246.38 86.36 180) (fields_autoplaced)
-    (effects (font (size 1.27 1.27)) (justify right bottom))
-  )
-  (label "IN" (at 165.1 156.21 0) (fields_autoplaced)
+  (label "1mADC_CH2" (at 222.25 88.9 0) (fields_autoplaced)
+    (effects (font (size 1.27 1.27)) (justify left bottom))
+  )
+  (label "CH2+" (at 271.78 88.9 0) (fields_autoplaced)
+    (effects (font (size 1.27 1.27)) (justify left bottom))
+  )
+  (label "IN" (at 165.1 154.94 0) (fields_autoplaced)
     (effects (font (size 1.27 1.27)) (justify left bottom))
   )
@@
     (effects (font (size 1.27 1.27)) (justify right bottom))
   )
-  (label "CH1-" (at 270.51 53.34 0) (fields_autoplaced)
-    (effects (font (size 1.27 1.27)) (justify left bottom))
-  )
-  (label "CH2+" (at 222.25 88.9 0) (fields_autoplaced)
-    (effects (font (size 1.27 1.27)) (justify left bottom))
-  )
   (label "5V_REG" (at 127 41.91 0) (fields_autoplaced)
     (effects (font (size 1.27 1.27)) (justify left bottom))
   )
-  (label "CH1-" (at 224.79 52.07 0) (fields_autoplaced)
-    (effects (font (size 1.27 1.27)) (justify left bottom))
-  )
   (label "1mADC_CH2" (at 158.75 74.93 0) (fields_autoplaced)
     (effects (font (size 1.27 1.27)) (justify left bottom))
   )
+  (label "~{IN}" (at 246.38 104.14 180) (fields_autoplaced)
+    (effects (font (size 1.27 1.27)) (justify right bottom))
+  )
   (label "CH2+" (at 266.7 142.24 0) (fields_autoplaced)
     (effects (font (size 1.27 1.27)) (justify left bottom))
@@
   (label "IN" (at 196.85 91.44 180) (fields_autoplaced)
     (effects (font (size 1.27 1.27)) (justify right bottom))
-  )
-  (label "CH2+" (at 222.25 101.6 0) (fields_autoplaced)
-    (effects (font (size 1.27 1.27)) (justify left bottom))
   )
   (symbol (lib_id "Device:C") (at 154.94 168.91 0) (unit 1)
@@
         (path "/485d57e1-9e59-4bdb-b543-f102996c1764"
           (reference "R9") (unit 1)
+        )
+      )
+    )
+  )
+  (symbol (lib_id "power:GNDA") (at 199.39 49.53 270) (unit 1)
+    (in_bom yes) (on_board yes) (dnp no) (fields_autoplaced)
+    (property "Reference" "#PWR017" (at 193.04 49.53 0)
+      (effects (font (size 1.27 1.27)) hide)
+    )
+    (property "Value" "GNDA" (at 195.58 50.165 90)
+      (effects (font (size 1.27 1.27)) (justify right))
+    )
+    (property "Footprint" "" (at 199.39 49.53 0)
+      (effects (font (size 1.27 1.27)) hide)
+    )
+    (property "Datasheet" "" (at 199.39 49.53 0)
+      (effects (font (size 1.27 1.27)) hide)
+    )
+    (pin "1")
+    (instances
+      (project "Fonte-de-corrente-SWLS_V0"
+        (path "/485d57e1-9e59-4bdb-b543-f102996c1764"
+          (reference "#PWR017") (unit 1)
         )
       )
@@
     )
   )
-  (symbol (lib_id "power:GNDA") (at 246.38 99.06 270) (unit 1)
-    (in_bom yes) (on_board yes) (dnp no) (fields_autoplaced)
-    (property "Reference" "#PWR019" (at 240.03 99.06 0)
-      (effects (font (size 1.27 1.27)) hide)
-    )
-    (property "Value" "GNDA" (at 242.57 99.695 90)
-      (effects (font (size 1.27 1.27)) (justify right))
-    )
-    (property "Footprint" "" (at 246.38 99.06 0)
-      (effects (font (size 1.27 1.27)) hide)
-    )
-    (property "Datasheet" "" (at 246.38 99.06 0)
-      (effects (font (size 1.27 1.27)) hide)
-    )
-    (pin "1")
-    (instances
-      (project "Fonte-de-corrente-SWLS_V0"
-        (path "/485d57e1-9e59-4bdb-b543-f102996c1764"
-          (reference "#PWR019") (unit 1)
-        )
-      )
-    )
-  )
   (symbol (lib_id "74xGxx:74AHC1G04") (at 151.13 180.34 0) (unit 1)
     (in_bom yes) (on_board yes) (dnp no)
@@
     )
   )
-  (symbol (lib_id "power:GNDA") (at 199.39 49.53 270) (unit 1)
-    (in_bom yes) (on_board yes) (dnp no) (fields_autoplaced)
-    (property "Reference" "#PWR017" (at 193.04 49.53 0)
-      (effects (font (size 1.27 1.27)) hide)
-    )
-    (property "Value" "GNDA" (at 195.58 50.165 90)
-      (effects (font (size 1.27 1.27)) (justify right))
-    )
-    (property "Footprint" "" (at 199.39 49.53 0)
-      (effects (font (size 1.27 1.27)) hide)
-    )
-    (property "Datasheet" "" (at 199.39 49.53 0)
-      (effects (font (size 1.27 1.27)) hide)
-    )
-    (pin "1")
-    (instances
-      (project "Fonte-de-corrente-SWLS_V0"
-        (path "/485d57e1-9e59-4bdb-b543-f102996c1764"
-          (reference "#PWR017") (unit 1)
-        )
-      )
-    )
-  )
   (symbol (lib_id "Device:R") (at 143.51 52.07 90) (unit 1)
     (in_bom yes) (on_board yes) (dnp no)
@@
         )
       )
+    )
+  )
+  (symbol (lib_id "power:GNDA") (at 246.38 86.36 270) (unit 1)
+    (in_bom yes) (on_board yes) (dnp no) (fields_autoplaced)
+    (property "Reference" "#PWR028" (at 240.03 86.36 0)
+      (effects (font (size 1.27 1.27)) hide)
+    )
+    (property "Value" "GNDA" (at 242.57 86.995 90)
+      (effects (font (size 1.27 1.27)) (justify right))
+    )
+    (property "Footprint" "" (at 246.38 86.36 0)
+      (effects (font (size 1.27 1.27)) hide)
+    )
+    (property "Datasheet" "" (at 246.38 86.36 0)
+      (effects (font (size 1.27 1.27)) hide)
+    )
+    (pin "1")
+    (instances
+      (project "Fonte-de-corrente-SWLS_V0"
+        (path "/485d57e1-9e59-4bdb-b543-f102996c1764"
+          (reference "#PWR028") (unit 1)
+        )
+      )

Commit message: Atualização do layout de PCB
Parts:
- removed SW1: SW_DIP_x01, Fonte-de-corrente-SWLS-complementar:Chave analógica, symbol Switch:SW_DIP_x01
- added SW1: SW_DPDT_x2, Fonte-de-corrente-SWLS-complementar:SW_100SP1T2B4M6QE, symbol Switch:SW_DPDT_x2
Connections:
- net +5V: now also SW1.1 (A)
- net GND: now also SW1.3 (C)
- net IN: now also SW1.2 (B)
Changed lines of the file:
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@@
   (junction (at 54.61 41.91) (diameter 0) (color 0 0 0 0)
   )
+  (junction (at 116.84 154.94) (diameter 0) (color 0 0 0 0)
+  )
   (junction (at 134.62 154.94) (diameter 0) (color 0 0 0 0)
   )
@@
   )
   (junction (at 50.8 49.53) (diameter 0) (color 0 0 0 0)
-  )
-  (junction (at 116.84 154.94) (diameter 0) (color 0 0 0 0)
   )
   (junction (at 151.13 46.99) (diameter 0) (color 0 0 0 0)
@@
     (stroke (width 0) (type dash))
   )
+  (wire (pts (xy 116.84 154.94) (xy 116.84 157.48))
+    (stroke (width 0) (type default))
+  )
   (polyline (pts (xy 135.89 48.26) (xy 135.89 44.45))
     (stroke (width 0) (type dash))
@@
         (path "/485d57e1-9e59-4bdb-b543-f102996c1764"
           (reference "#PWR017") (unit 1)
+        )
+      )
+    )
+  )
+  (symbol (lib_name "+5VD_1") (lib_id "power:+5VD") (at 119.38 167.64 180) (unit 1)
+    (in_bom yes) (on_board yes) (dnp no) (fields_autoplaced)
+    (property "Reference" "#PWR019" (at 119.38 163.83 0)
+      (effects (font (size 1.27 1.27)) hide)
+    )
+    (property "Value" "+5VDC" (at 119.38 172.72 0)
+      (effects (font (size 1.27 1.27)))
+    )
+    (property "Footprint" "" (at 119.38 167.64 0)
+      (effects (font (size 1.27 1.27)) hide)
+    )
+    (property "Datasheet" "" (at 119.38 167.64 0)
+      (effects (font (size 1.27 1.27)) hide)
+    )
+    (pin "1")
+    (instances
+      (project "Fonte-de-corrente-SWLS_V0"
+        (path "/485d57e1-9e59-4bdb-b543-f102996c1764"
+          (reference "#PWR019") (unit 1)
         )
       )
@@
     )
   )
+  (symbol (lib_id "Switch:SW_DPDT_x2") (at 116.84 162.56 270) (unit 1)
+    (in_bom yes) (on_board yes) (dnp no) (fields_autoplaced)
+    (property "Reference" "SW1" (at 120.65 161.925 90)
+      (effects (font (size 1.27 1.27)) (justify left))
+    )
+    (property "Value" "SW_DPDT_x2" (at 120.65 164.465 90)
+      (effects (font (size 1.27 1.27)) (justify left))
+    )
+    (property "Footprint" "Fonte-de-corrente-SWLS-complementar:SW_100SP1T2B4M6QE" (at 116.84 162.56 0)
+      (effects (font (size 1.27 1.27)) hide)
+    )
+    (property "Datasheet" "https://sten-eswitch-13110800-production.s3.amazonaws.com/system/asset/product_line/data_sheet/129/100.pdf" (at 116.84 162.56 0)
+      (effects (font (size 1.27 1.27)) hide)
+    )
+    (property "Numero do produto" "100SP1T2B4M6QE" (at 116.84 162.56 90)
+      (effects (font (size 1.27 1.27)) hide)
+    )
+    (pin "1")
+    (pin "2")
+    (pin "3")
+    (pin "4")
+    (pin "5")
+    (pin "6")
+    (instances
+      (project "Fonte-de-corrente-SWLS_V0"
+        (path "/485d57e1-9e59-4bdb-b543-f102996c1764"
+          (reference "SW1") (unit 1)
+        )
+      )
+    )
+  )
   (symbol (lib_name "LM4810_1") (lib_id "Amplifier_Audio:LM4810") (at 212.09 40.64 0) (unit 1)
     (in_bom yes) (on_board yes) (dnp no)
@@
     )
   )
-  (symbol (lib_name "GND_2") (lib_id "power:GND") (at 116.84 170.18 0) (unit 1)
-    (in_bom yes) (on_board yes) (dnp no) (fields_autoplaced)
-    (property "Reference" "#PWR015" (at 116.84 176.53 0)
-      (effects (font (size 1.27 1.27)) hide)
-    )
-    (property "Value" "GND" (at 116.84 175.26 0)
-      (effects (font (size 1.27 1.27)))
-    )
-    (property "Footprint" "" (at 116.84 170.18 0)
-      (effects (font (size 1.27 1.27)) hide)
-    )
-    (property "Datasheet" "" (at 116.84 170.18 0)
+  (symbol (lib_name "GND_2") (lib_id "power:GND") (at 114.3 167.64 0) (unit 1)
+    (in_bom yes) (on_board yes) (dnp no) (fields_autoplaced)
+    (property "Reference" "#PWR015" (at 114.3 173.99 0)
+      (effects (font (size 1.27 1.27)) hide)
+    )
+    (property "Value" "GND" (at 114.3 172.72 0)
+      (effects (font (size 1.27 1.27)))
+    )
+    (property "Footprint" "" (at 114.3 167.64 0)
+      (effects (font (size 1.27 1.27)) hide)
+    )
+    (property "Datasheet" "" (at 114.3 167.64 0)
       (effects (font (size 1.27 1.27)) hide)
     )
@@
         )
       )
-    )
-  )
-  (symbol (lib_id "Switch:SW_DIP_x01") (at 116.84 162.56 90) (unit 1)
-    (in_bom yes) (on_board yes) (dnp no) (fields_autoplaced)
-    (property "Reference" "SW1" (at 120.65 161.2899 90)
-      (effects (font (size 1.27 1.27)) (justify right))
-    )
-    (property "Value" "SW_DIP_x01" (at 120.65 163.8299 90)
-      (effects (font (size 1.27 1.27)) (justify right))
-    )
-    (property "Footprint" "Fonte-de-corrente-SWLS-complementar:Chave analógica" (at 116.84 162.56 0)
-      (effects (font (size 1.27 1.27)) hide)
-    )
-    (property "Datasheet" "https://br.mouser.com/datasheet/2/445/418117270901-3086928.pdf" (at 116.84 162.56 0)
-      (effects (font (size 1.27 1.27)) hide)
-    )
-    (property "Numero do Produto" "418117270901" (at 116.84 162.56 90)
-      (effects (font (size 1.27 1.27)) hide)
-    )
-    (pin "1")
-    (pin "2")
-    (instances
-      (project "Fonte-de-corrente-SWLS_V0"
-        (path "/485d57e1-9e59-4bdb-b543-f102996c1764"
-          (reference "SW1") (unit 1)
-        )
-      )
