File: pcb/cad/Fonte-de-corrente-SWLS_V0/Fonte-de-corrente-SWLS_V0.kicad_pcb (KiCad board)
At the start: 2 copper layers, 59.9 x 38 mm, 33 parts, among them J2 LEMO FFA.0S, J3 LEMO FFA.0S, J4 Barrel_Jack_Switch, SW1 SW_DPDT_x2, U1 LM78L05, U2 LT3080xST, U3 LT3092xST, U4 LT3092xST, U5 74AHC1G04, U6 TS5A21366, U7 TS5A21366, U8 TS5A21366, U9 TS5A21366

Commit message: Atualização da ultima versão da PCB e esquemático
Parts:
- C6, C7, C8, C9: footprint Capacitor_SMD:C_0805_2012Metric -> Capacitor_SMD:C_1206_3216Metric
- moved R4 2.22 mm to (47.7, 44.4)
- moved U3 2.22 mm to (41.0, 47.0)
- moved R8 2.22 mm to (47.7, 47.0)
- moved R6 1.85 mm to (47.5, 49.6)
- moved R9 1.58 mm to (47.5, 55.2)
- moved R7 1.58 mm to (47.5, 57.7)
- moved U4 1.58 mm to (41.1, 55.2)
- moved R5 1.40 mm to (47.5, 52.7)
Routing:
- net GNDA: track 9.24 -> 34.7 mm
- net GND: track 32.6 -> 35.6 mm
- net /CH1-: track 22.9 -> 24.8 mm
- net /~{IN}: track 96.5 -> 98.0 mm
- net /1mADC_CH1: track 22.6 -> 24.1 mm
- net /5V_REG: track 55.5 -> 54.5 mm
- net +5V: track 137.0 -> 136.1 mm
- net /CH2-: track 22.6 -> 23.3 mm
- net /1mADC_CH2: track 25.6 -> 26.2 mm
